File: hardware/main/connector.kicad_sch (KiCad schematic)
At the start: 27 parts, among them J11 TF-01A, J3 Conn_01x04, J4 Conn_01x04, J5 Conn_01x04, J6 Conn_01x04, J7 Conn_01x10, J7b Conn_01x08, J8 Conn_01x06, J9 Conn_01x04

Commit message: hardware: 48 erreurs ERC traitees, 22 points de test poses, VBAT_SENSE retire de J8.5
Les rapports ERC precedents portaient « Report includes: Warnings » : les
erreurs en etaient exclues a l'export et le resume affichait « Errors 0 ».
Elles etaient donc presentes depuis le debut et je ne les ai pas vues — il faut
exporter avec les erreurs incluses.

48 erreurs, trois familles, toutes des faux positifs au sens electrique mais
qu'il faut declarer sinon l'ERC reste inexploitable :

1. power_pin_not_driven (14) : le projet n'utilise aucun symbole d'alimentation,
   les rails sont des global labels, et KiCad exige qu'un net « power input »
   soit pilote par une pin « power output ». Nine PWR_FLAG poses, un par rail
   (GND, VSYS, VBAT, VBAT-, 3V3_D, 3V3_A, 5V, 5V_BOOST, 5V_USB).
2. pin_not_connected (29) : broches volontairement libres — paires SuperSpeed et
   SBU de l'USB-C (design USB 2.0), UART0 et IO35-37 de l'ESP32 (reserves a la
   PSRAM octale), GPIO du PCM5122, interruptions de l'IMU, reserves de
   connecteurs, drains communs du FS8205. Marqueurs no_connect.
3. divers (5) : label GND orphelin hors page (122, 228.81 — la page fait
   210 mm de haut) supprime ; C1_AV/C2_DV/C3_CP renommes C_AVDD/C_DVDD/C_CPVDD
   (KiCad lit « C1_AV » comme un prefixe suivi de « 1_AV », donc non annote) ;
   OUT_11 du bq24075 passee en passive (les deux broches sont la meme sortie).

Points de test : les 22 valides sont poses, chacun relie par un fil court a un
global label (le routeur les placera ou ils sont accessibles). 22/22 verifies
sur leur net. Trois nets anonymes nommes au passage : BQ_ISET, BQ_CHG,
BOOST_FB. Avec les 4 existants, 26 points de test.

VBAT_SENSE retire de J8.5 : noeud ADC haute impedance (1M // 1M) sorti dans un
cable, sans usage cote face avant depuis que les analogiques passent par
l'ADS7830. Broche marquee non connectee.

CORRECTION D'OUTIL : tools/kicad_netlist.py comptait PWR_FLAG comme un nom de
net, ce qui faisait fusionner les neuf rails en un seul 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
Parts:
- added TP_WS2812: TestPoint, TestPoint:TestPoint_Pad_D1.5mm, symbol Connector:TestPoint
Connections:
- net WS2812_DATA: now also TP_WS2812.1
- net VBAT_SENSE: no longer names the net of J8.5 (Pin_5)
- no-connect marks 0 -> 6
Changed lines of the file:
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@@
 	(wire
 		(pts
-			(xy 91.44 57.15) (xy 82.44 57.15)
-		)
-		(stroke
-			(width 0)
-			(type default)
-		)
-	)
-	(wire
-		(pts
 			(xy 66.04 109.22) (xy 72.39 109.22)
 		)
@@
 		)
 	)
-	(global_label "VBAT_SENSE"
-		(shape input)
-		(at 82.44 57.15 180)
-		(fields_autoplaced yes)
-		(effects
-			(font
-				(size 1.27 1.27)
-			)
-			(justify right)
-		)
-		(property "Intersheetrefs" "${INTERSHEET_REFS}"
-			(at 5.1791 16.51 0)
-			(hide yes)
-			(show_name no)
-			(do_not_autoplace no)
-			(effects
-				(font
-					(size 1.27 1.27)
-				)
-				(justify right)
-			)
-		)
-	)
 	(global_label "GND"
 		(shape input)
@@
 			)
 		)
+	)
+	(no_connect
+		(at 260.35 43.18)
+	)
+	(no_connect
+		(at 260.35 45.72)
+	)
+	(no_connect
+		(at 91.44 59.69)
+	)
+	(no_connect
+		(at 44.45 132.08)
+	)
+	(no_connect
+		(at 134.62 160.02)
+	)
+	(no_connect
+		(at 91.44 57.15)
+	)
+	(symbol
+		(lib_id "Connector:TestPoint")
+		(at 17.78 191.77 0)
+		(unit 1)
+		(body_style 1)
+		(exclude_from_sim no)
+		(in_bom yes)
+		(on_board yes)
+		(in_pos_files yes)
+		(dnp no)
+		(property "Reference" "TP_WS2812"
+			(at 20.32 190.5 0)
+			(show_name no)
+			(do_not_autoplace no)
+			(effects
+				(font
+					(size 1.27 1.27)
+				)
+			)
+		)
+		(property "Value" "TestPoint"
+			(at 20.32 193.04000000000002 0)
+			(show_name no)
+			(do_not_autoplace no)
+			(effects
+				(font
+					(size 1.27 1.27)
+				)
+			)
+		)
+		(property "Footprint" "TestPoint:TestPoint_Pad_D1.5mm"
+			(at 17.78 191.77 0)
+			(hide yes)
+			(show_name no)
+			(do_not_autoplace no)
+			(effects
+				(font
+					(size 1.27 1.27)
+				)
+			)
+		)
+		(property "Datasheet" ""
+			(at 17.78 191.77 0)
+			(hide yes)
+			(show_name no)
+			(do_not_autoplace no)
+			(effects
+				(font
+					(size 1.27 1.27)
+				)
+			)
+		)
+		(property "Description" "Point de test WS2812_DATA — voir docs/pcb/03-validation-qualite.md"
+			(at 17.78 191.77 0)
+			(hide yes)
+			(show_name no)
+			(do_not_autoplace no)
+			(effects
+				(font
+					(size 1.27 1.27)
+				)
+			)
+		)
+		(pin "1"
+		)
+		(instances
+			(project "blackbox"
+				(path "/49e0257f-ff47-4890-a1ac-89438fa62044/51b01d3e-87dc-456c-a96b-c77ebbca5dc9"
+					(reference "TP_WS2812")
+					(unit 1)
+				)
+			)
+		)
+	)
+	(wire
+		(pts
+			(xy 17.78 191.77) (xy 17.78 196.85000000000002)
+		)
+		(stroke
+			(width 0)
+			(type default)
+		)
+	)
+	(global_label "WS2812_DATA"
+		(shape input)
+		(at 17.78 196.85000000000002 270)
+		(fields_autoplaced yes)
+		(effects
+			(font
+				(size 1.27 1.27)
+			)
+			(justify left)
+		)
+		(property "Intersheetrefs" "${INTERSHEET_REFS}"
+			(at 29.21 196.85000000000002 0)
+			(hide yes)
+			(show_name no)
+			(do_not_autoplace no)
+			(effects
+				(font
+					(size 1.27 1.27)
+				)
+				(justify left)
+			)
+		)

Commit message: datasheets: ATtiny1616, reference documentaire non inventee
Parts:
- added J13: Conn_01x04, Connector_JST:JST_SH_BM04B-SRSS-TB_1x04-1MP_P1.00mm_Vertical, symbol Connector_Generic:Conn_01x04
- added R23, R24: 10k, Resistor_SMD:R_0402_1005Metric, symbol Device:R
Connections:
- net 3V3_D: now also J13.2 (Pin_2)
- net GND: now also J13.1 (Pin_1), R23.2, R24.2
- net I2C_SCL: now also J13.4 (Pin_4)
- net I2C_SDA: now also J13.3 (Pin_3)
- net BTN1: now reaches J8.5 (Pin_5)
- net BTN1: now also R23.1
- net BTN2: now reaches J8.6 (Pin_6)
- net BTN2: now also R24.1
- no-connect marks 6 -> 4
Other:
- moved on the sheet: TP_WS2812
