File: hardware/main/imu.kicad_sch (KiCad schematic)
At the start: 3 parts, among them U11 LSM6DSOXTR

Commit message: hardware: 48 erreurs ERC traitees, 22 points de test poses, VBAT_SENSE retire de J8.5
Les rapports ERC precedents portaient « Report includes: Warnings » : les
erreurs en etaient exclues a l'export et le resume affichait « Errors 0 ».
Elles etaient donc presentes depuis le debut et je ne les ai pas vues — il faut
exporter avec les erreurs incluses.

48 erreurs, trois familles, toutes des faux positifs au sens electrique mais
qu'il faut declarer sinon l'ERC reste inexploitable :

1. power_pin_not_driven (14) : le projet n'utilise aucun symbole d'alimentation,
   les rails sont des global labels, et KiCad exige qu'un net « power input »
   soit pilote par une pin « power output ». Nine PWR_FLAG poses, un par rail
   (GND, VSYS, VBAT, VBAT-, 3V3_D, 3V3_A, 5V, 5V_BOOST, 5V_USB).
2. pin_not_connected (29) : broches volontairement libres — paires SuperSpeed et
   SBU de l'USB-C (design USB 2.0), UART0 et IO35-37 de l'ESP32 (reserves a la
   PSRAM octale), GPIO du PCM5122, interruptions de l'IMU, reserves de
   connecteurs, drains communs du FS8205. Marqueurs no_connect.
3. divers (5) : label GND orphelin hors page (122, 228.81 — la page fait
   210 mm de haut) supprime ; C1_AV/C2_DV/C3_CP renommes C_AVDD/C_DVDD/C_CPVDD
   (KiCad lit « C1_AV » comme un prefixe suivi de « 1_AV », donc non annote) ;
   OUT_11 du bq24075 passee en passive (les deux broches sont la meme sortie).

Points de test : les 22 valides sont poses, chacun relie par un fil court a un
global label (le routeur les placera ou ils sont accessibles). 22/22 verifies
sur leur net. Trois nets anonymes nommes au passage : BQ_ISET, BQ_CHG,
BOOST_FB. Avec les 4 existants, 26 points de test.

VBAT_SENSE retire de J8.5 : noeud ADC haute impedance (1M // 1M) sorti dans un
cable, sans usage cote face avant depuis que les analogiques passent par
l'ADS7830. Broche marquee non connectee.

CORRECTION D'OUTIL : tools/kicad_netlist.py comptait PWR_FLAG comme un nom de
net, ce qui faisait fusionner les neuf rails en un seul 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
Connections:
- no-connect marks 0 -> 4
Changed lines of the file:
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@@
 		)
 	)
+	(no_connect
+		(at 135.89 87.63)
+	)
+	(no_connect
+		(at 168.91 92.71)
+	)
+	(no_connect
+		(at 168.91 90.17)
+	)
+	(no_connect
+		(at 168.91 87.63)
+	)
 )
