File: hardware/main/power.kicad_sch (KiCad schematic)
At the start: 57 parts, among them J12 Interrupteur, J14 USB Cote 2, J2 Batterie 18650, Q1 AO3401A, Q2 2N7002, U10 FS8205, U5 AP2112M-3.3, U6 AP2112K-3.3, U7 MT3608, U8 BQ24075RGTR, U9 DW01A

Commit message: power: R20 100k -> 2k2 (courant de contact pour SW3 E-Switch RR1, contacts argent)
Parts:
- R20: value 100k -> 2k2
Changed lines of the file:
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@@
 			)
 		)
-		(property "Value" "100k"
+		(property "Value" "2k2"
 			(at 165.608 69.596 0)
 			(show_name no)
@@
 			)
 		)
-		(property "Description" "Pull-down EN_SYS : coupe les rails si J12 est ouvert ou debranche"
+		(property "Description" "Pull-down EN_SYS : coupe les rails si J12 est ouvert ou debranche. 2,2 k (2026-09-27) : ~1,5-2,5 mA dans le contact argent de SW3 (E-Switch RR1) quand la box est allumee"
 			(at 161.29 67.31 0)
 			(hide yes)

Commit message: power: C_IN 4,7 uF 25 V X7R 0805 (YAGEO C354262), au lieu de 10 V 0603
Parts:
- C_IN: footprint Capacitor_SMD:C_0603_1608Metric -> Capacitor_SMD:C_0805_2012Metric
Changed lines of the file:
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@@
 			)
 		)
-		(property "Footprint" "Capacitor_SMD:C_0603_1608Metric"
+		(property "Footprint" "Capacitor_SMD:C_0805_2012Metric"
 			(at 190.1952 45.72 0)
 			(hide yes)

Commit message: power: C_IN 4,7 uF 25 V X5R 0603 (Samsung CL10A475KA8NQNC, C69335), empreinte 0603 conservee
Parts:
- C_IN: footprint Capacitor_SMD:C_0805_2012Metric -> Capacitor_SMD:C_0603_1608Metric
Changed lines of the file:
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@@
 			)
 		)
-		(property "Footprint" "Capacitor_SMD:C_0805_2012Metric"
+		(property "Footprint" "Capacitor_SMD:C_0603_1608Metric"
 			(at 190.1952 45.72 0)
 			(hide yes)
